Commit message: mods for hydro

File: r2_description/robots/r2.urdf.xacro (robot description, xacro)
@@ -1,12 +1,15 @@
 <?xml version="1.0" ?>
-<robot name="r2">
+<robot name="r2" xmlns:controller="http://playerstage.sourceforge.net/gazebo/xmlschema/#controller"
+			xmlns:interface="http://playerstage.sourceforge.net/gazebo/xmlschema/#interface"
+			xmlns:sensor="http://playerstage.sourceforge.net/gazebo/xmlschema/#sensor"
+			xmlns:xacro="http://playerstage.sourceforge.net/gazebo/xmlschema/#interface">
   <property name="robot_name" value= "/r2/" />
-  <include filename="$(find r2_description)/urdf/r2.common.xacro" />
-  <include filename="$(find r2_description)/urdf/r2.base.xacro" />
-  <include filename="$(find r2_description)/urdf/r2.body.xacro" />
-  <include filename="$(find r2_description)/urdf/r2.head.xacro" />
-  <include filename="$(find r2_description)/urdf/r2.left_arm.xacro" />
-  <include filename="$(find r2_description)/urdf/r2.left_hand.xacro" />
-  <include filename="$(find r2_description)/urdf/r2.right_arm.xacro" />
-  <include filename="$(find r2_description)/urdf/r2.right_hand.xacro" />
+  <xacro:include filename="$(find r2_description)/urdf/r2.common.xacro" />
+  <xacro:include filename="$(find r2_description)/urdf/r2.base.xacro" />
+  <xacro:include filename="$(find r2_description)/urdf/r2.body.xacro" />
+  <xacro:include filename="$(find r2_description)/urdf/r2.head.xacro" />
+  <xacro:include filename="$(find r2_description)/urdf/r2.left_arm.xacro" />
+  <xacro:include filename="$(find r2_description)/urdf/r2.left_hand.xacro" />
+  <xacro:include filename="$(find r2_description)/urdf/r2.right_arm.xacro" />
+  <xacro:include filename="$(find r2_description)/urdf/r2.right_hand.xacro" />
 </robot>

File: r2_description/urdf/r2.body.xacro (robot description, xacro)
@@ -1,6 +1,6 @@
 <?xml version="1.0"?>
 <robot>
-  <property name="waist_j0_damping" value= "10.0" />
-  <property name="waist_j0_friction" value= "0.0" />
+  <property name="waist_j0_damping" value= "20.0" />
+  <property name="waist_j0_friction" value= "1.0" />
   <joint name="${robot_name}waist/joint0" type="revolute">
     <parent link="${robot_name}robot_base"/>

File: r2_description/urdf/r2.head.xacro (robot description, xacro)
@@ -1,9 +1,9 @@
 <?xml version="1.0"?>
 <robot>
-  <property name="neck_j0_damping" value= "10.0" />
+  <property name="neck_j0_damping" value= "1.0" />
   <property name="neck_j0_friction" value= "0.0" />
-  <property name="neck_j1_damping" value= "10.0" />
+  <property name="neck_j1_damping" value= "1.0" />
   <property name="neck_j1_friction" value= "0.0" />
-  <property name="neck_j2_damping" value= "10.0" />
+  <property name="neck_j2_damping" value= "1.0" />
   <property name="neck_j2_friction" value= "0.0" />
   <property name="effort_limit" value= "10000.0" />

File: r2_description/urdf/r2.left_arm.xacro (robot description, xacro)
@@ -167,5 +167,5 @@
         <origin xyz="-0.004064   0.000000152908   -0.00092202"/>
         <mass value="0.1165732391"/>
-        <inertia ixx="0.00005765"  ixy="0.00000000004360"  ixz="0.00000175876"  iyy="0.0000169438359087"  iyz="0.000000054430975458"  izz="0.000044188587603"/>
+        <inertia ixx="0.1"  ixy="0.0"  ixz="0.0"  iyy="0.1"  iyz="0.0"  izz="0.1"/>
     </inertial>
   </link>
@@ -181,6 +181,6 @@
     <inertial>
         <origin xyz="-0.00090932   -0.0253746  0.067564     "/>
-        <mass value="1.1884120094"/>
-        <inertia ixx="0.0044481227"  ixy="0.0003716524"  ixz="0.0001024239"  iyy="0.0030141884"  iyz="0.000101546"  izz="0.001992876"/>
+        <mass value="0.1"/>
+        <inertia ixx="0.1"  ixy="0.0"  ixz="0.0"  iyy="0.1"  iyz="0.0"  izz="0.1"/>
     </inertial>
   </link>
@@ -205,6 +205,6 @@
     <inertial>
         <origin xyz="0.067564   -0.0253746   -0.00090932"/>
-        <mass value="1.1884120094"/>
-        <inertia ixx="0.001992876"  ixy="0.000101546"  ixz="0.0001024239"  iyy="0.0030141884"  iyz="0.0003716524"  izz="0.0044481227"/>
+        <mass value="1.1"/>
+        <inertia ixx="0.1"  ixy="0.0"  ixz="0.0"  iyy="0.1"  iyz="0.0"  izz="0.1"/>
     </inertial>
   </link>

File: r2_description/urdf/r2.right_arm.xacro (robot description, xacro)
@@ -167,5 +167,5 @@
         <origin xyz="0.00092202 -0.004064 0.000000152908"/>
         <mass value="0.1165732391"/>
-        <inertia ixx=".0000169438359087"  ixy=".000000054430975458"  ixz="-.000000000043603308297"  iyy=".000044188587603"  iyz="-.00000175876431453"  izz=".00005765"/>
+       <inertia ixx="0.1"  ixy="0.0"  ixz="0.0"  iyy="0.1"  iyz="0.0"  izz="0.1"/>
     </inertial>
   </link>
@@ -181,6 +181,6 @@
     <inertial>
         <origin xyz="0.067564 0.00090932 0.0253746"/>
-        <mass value="1.1884120094"/>
-        <inertia ixx="0.001992876"  ixy="-0.0001024239"  ixz="-0.000101546"  iyy="0.0044481227"  iyz="0.0003716524"  izz="0.0030141884"/>
+        <mass value="0.1"/>
+       <inertia ixx="0.1"  ixy="0.0"  ixz="0.0"  iyy="0.1"  iyz="0.0"  izz="0.1"/>
     </inertial>
   </link>
@@ -204,6 +204,6 @@
     </collision>
     <inertial>
-      <mass value="0.1"/>
-      <inertia ixx=".0010" ixy="0.0" ixz="0.0" iyy=".0010" iyz="0.0" izz=".0010"/>
+        <mass value="1.1"/>
+        <inertia ixx="0.1"  ixy="0.0"  ixz="0.0"  iyy="0.1"  iyz="0.0"  izz="0.1"/>
     </inertial>
   </link>
