Commit message: added legs moveit package and renamed things a bit

File: r2_description/robots/r2_fullbody.urdf.xacro (robot description, xacro)
@@ -4,7 +4,7 @@
        xmlns:interface="http://playerstage.sourceforge.net/gazebo/xmlschema/#interface"
        xmlns:xacro="http://playerstage.sourceforge.net/gazebo/xmlschema/#interface"
-       name="r2c_full_body" >
+       name="r2_fullbody" >
   <link name="world"/>
-  <property name="robot_name" value= "/r2/" />
+  <property name="robot_name" value= "r2/" />
 <!--  transforms in first joint don't seem to work properly-->
   <joint name="${robot_name}fixed/world/robot_world" type="fixed">
@@ -13,7 +13,4 @@
     <origin rpy="0 0 0.0" xyz="0.0 0.0 0.0"/>
   </joint>
-  <xacro:include filename="$(find r2_description)/robots/r2c_full_body_no_world.urdf.xacro" />
-  <xacro:robot_base_origin>
-    <origin xyz="0 0 1.4" rpy="0 0 0" />
-  </xacro:robot_base_origin>
+  <xacro:include filename="$(find r2_description)/robots/r2_fullbody_no_world.urdf.xacro" />
 </robot>

File: r2_description/robots/r2_fullbody_no_world.urdf.xacro (robot description, xacro)
@@ -1,14 +1,12 @@
 <?xml version="1.0" ?>
-<robot name="r2c_full_body" xmlns:xacro="http://playerstage.sourceforge.net/gazebo/xmlschema/#interface">
-  <property name="robot_name" value= "/r2/" />
-  <non_visual_link name="${robot_name}robot_world"/>
-  <xacro:macro name="robot_base_origin" params="*origin">
-    <joint name="${robot_name}fixed/robot_world/robot_base" type="fixed">
+<robot name="r2" xmlns:xacro="http://playerstage.sourceforge.net/gazebo/xmlschema/#interface">
+  <property name="robot_name" value= "r2/" />
+  <link name="${robot_name}robot_world"/>
+  <joint name="${robot_name}fixed/robot_world/robot_base" type="fixed">
       <parent link="${robot_name}robot_world"/>
       <child link="${robot_name}robot_base"/>
-      <xacro:insert_block name="origin" />
-    </joint>
-  </xacro:macro>
-  <non_visual_link name="${robot_name}robot_base"/>
+      <origin rpy="0 3.14159 1.57079" xyz="0.255 0.9 1.365"/>
+  </joint>
+  <link name="${robot_name}robot_base"/>
   <joint name="${robot_name}fixed/robot_base/leg_stand_connection" type="fixed">
     <parent link="${robot_name}robot_base"/>
@@ -24,8 +22,8 @@
   <xacro:include filename="$(find r2_description)/urdf/r2.right_arm.xacro" />
   <xacro:include filename="$(find r2_description)/urdf/r2.right_hand.xacro" />
-  <xacro:include filename="$(find r2_description)/urdf/r2c_legs/r2c_legs.pelvis.xacro" />
-  <xacro:include filename="$(find r2_description)/urdf/r2c_legs/r2c_legs.left_leg.xacro" />
-  <xacro:include filename="$(find r2_description)/urdf/r2c_legs/r2c_legs.left_foot.xacro" />
-  <xacro:include filename="$(find r2_description)/urdf/r2c_legs/r2c_legs.right_leg.xacro" />
-  <xacro:include filename="$(find r2_description)/urdf/r2c_legs/r2c_legs.right_foot.xacro" />
+  <xacro:include filename="$(find r2_description)/urdf/r2_legs/r2_legs.pelvis.xacro" />
+  <xacro:include filename="$(find r2_description)/urdf/r2_legs/r2_legs.left_leg.xacro" />
+  <xacro:include filename="$(find r2_description)/urdf/r2_legs/r2_legs.left_foot.xacro" />
+  <xacro:include filename="$(find r2_description)/urdf/r2_legs/r2_legs.right_leg.xacro" />
+  <xacro:include filename="$(find r2_description)/urdf/r2_legs/r2_legs.right_foot.xacro" />
 </robot>

File: r2_description/urdf/r2_legs/r2_legs.left_foot.xacro (robot description, xacro)
@@ -19,5 +19,5 @@
     <visual>
       <geometry>
-        <mesh filename="package://r2_description/meshes/r2c_legs/r2cl_foot.dae"/>
+        <mesh filename="package://r2_description/meshes/r2_legs/r2cl_foot.dae"/>
       </geometry>
       <origin rpy="0 0 0" xyz="0 0 0"/>
@@ -25,5 +25,5 @@
     <collision>
       <geometry>
-        <mesh filename="package://r2_description/meshes/r2c_legs/r2cl_foot.dae"/>
+        <mesh filename="package://r2_description/meshes/r2_legs/r2cl_foot.dae"/>
       </geometry>
       <origin rpy="0 0 0" xyz="0 0 0"/>
@@ -82,9 +82,9 @@
     <inertial>
       <mass value="0.16268"/>
-      <inertia ixx="0.001" ixy="0.0" ixz="0.0" iyy="0.001" iyz="0.0" izz="0.001"/>
+      <inertia ixx="0.1" ixy="0.0" ixz="0.0" iyy="0.1" iyz="0.0" izz="0.1"/>
     </inertial>
     <visual>
       <geometry>
-        <mesh filename="package://r2_description/meshes/r2c_legs/r2cl_foot_jaw1.dae"/>
+        <mesh filename="package://r2_description/meshes/r2_legs/r2cl_foot_jaw1.dae"/>
       </geometry>
       <origin rpy="0 0 0" xyz="0 0 0"/>
@@ -92,5 +92,5 @@
     <collision>
       <geometry>
-        <mesh filename="package://r2_description/meshes/r2c_legs/r2cl_foot_jaw1.dae"/>
+        <mesh filename="package://r2_description/meshes/r2_legs/r2cl_foot_jaw1.dae"/>
       </geometry>
       <origin rpy="0 0 0" xyz="0 0 0"/>
@@ -100,9 +100,9 @@
     <inertial>
       <mass value="0.16268"/>
-      <inertia ixx="0.001" ixy="0.0" ixz="0.0" iyy="0.001" iyz="0.0" izz="0.001"/>
+      <inertia ixx="0.1" ixy="0.0" ixz="0.0" iyy="0.1" iyz="0.0" izz="0.1"/>
     </inertial>
     <visual>
       <geometry>
-        <mesh filename="package://r2_description/meshes/r2c_legs/r2cl_foot_jaw2.dae"/>
+        <mesh filename="package://r2_description/meshes/r2_legs/r2cl_foot_jaw2.dae"/>
       </geometry>
       <origin rpy="0 0 0" xyz="0 0 0"/>
@@ -110,5 +110,5 @@
     <collision>
       <geometry>
-        <mesh filename="package://r2_description/meshes/r2c_legs/r2cl_foot_jaw2.dae"/>
+        <mesh filename="package://r2_description/meshes/r2_legs/r2cl_foot_jaw2.dae"/>
       </geometry>
       <origin rpy="0 0 0" xyz="0 0 0"/>

File: r2_description/urdf/r2_legs/r2_legs.left_leg.xacro (robot description, xacro)
@@ -51,14 +51,13 @@
     <dynamics damping="${left_leg_j0_damping}" friction="${left_leg_j0_friction}" />
     <limit effort="330.0" lower="-4.71239" upper="4.71239" velocity="1.0"/>
-    <traits spring_k="2.5"   />
   </joint>
   <link name="${robot_name}left_hip_roll">
     <inertial>
       <mass value="2.33931"/>
-      <inertia ixx="0.02547" ixy="0.00297" ixz="-0.00847" iyy="0.02956" iyz="0.00636" izz="0.01148"/>
-    </inertial>
-    <visual>
-      <geometry>
-        <mesh filename="package://r2_description/meshes/r2c_legs/r2cl_ext_bone3.dae"/>
+      <inertia ixx="0.1" ixy="0.00" ixz="0.0" iyy="0.1" iyz="0.0" izz="0.1"/>
+    </inertial>
+    <visual>
+      <geometry>
+        <mesh filename="package://r2_description/meshes/r2_legs/r2cl_ext_bone3.dae"/>
       </geometry>
       <origin rpy="0 0 0" xyz="0.0 0.0 0.0"/>
@@ -66,5 +65,5 @@
     <collision>
       <geometry>
-        <mesh filename="package://r2_description/meshes/r2c_legs/r2cl_ext_bone3.dae"/>
+        <mesh filename="package://r2_description/meshes/r2_legs/r2cl_ext_bone3.dae"/>
       </geometry>
       <origin rpy="0 0 0" xyz="0.0 0.0 0.0"/>
@@ -78,20 +77,19 @@
     <dynamics damping="${left_leg_j1_damping}" friction="${left_leg_j1_friction}" />
     <limit effort="330.0" lower="-1.483" upper="1.27" velocity="1.0"/>
-    <traits spring_k="2.5"   />
   </joint>
   <link name="${robot_name}left_hip_pitch">
     <inertial>
       <mass value="4.78221"/>
-      <inertia ixx="0.01671" ixy="0.02240" ixz="-0.00120" iyy="0.07877" iyz="0.00049" izz="0.08739"/>
-    </inertial>
-    <visual>
-      <geometry>
-        <mesh filename="package://r2_description/meshes/r2c_legs/r2cl_ext_bone1.dae"/>
-      </geometry>
-      <origin rpy="0 0 0" xyz="0 0 0"/>
-    </visual>
-    <collision>
-      <geometry>
-        <mesh filename="package://r2_description/meshes/r2c_legs/r2cl_ext_bone1.dae"/>
+      <inertia ixx="0.1" ixy="0.00" ixz="0.0" iyy="0.1" iyz="0.0" izz="0.1"/>
+    </inertial>
+    <visual>
+      <geometry>
+        <mesh filename="package://r2_description/meshes/r2_legs/r2cl_ext_bone1.dae"/>
+      </geometry>
+      <origin rpy="0 0 0" xyz="0 0 0"/>
+    </visual>
+    <collision>
+      <geometry>
+        <mesh filename="package://r2_description/meshes/r2_legs/r2cl_ext_bone1.dae"/>
       </geometry>
       <origin rpy="0 0 0" xyz="0 0 0"/>
@@ -105,20 +103,19 @@
     <dynamics damping="${left_leg_j2_damping}" friction="${left_leg_j2_friction}" />
     <limit effort="330.0" lower="-4.71239" upper="4.71239" velocity="1.0"/>
-    <traits spring_k="2.5"   />
   </joint>
   <link name="${robot_name}left_upper_leg">
     <inertial>
       <mass value="3.73407"/>
-      <inertia ixx="0.05967" ixy="-0.00299" ixz="0.00939" iyy="0.05554" iyz="0.01276" izz="0.01370"/>
-    </inertial>
-    <visual>
-      <geometry>
-        <mesh filename="package://r2_description/meshes/r2c_legs/r2cl_ext_bone2.dae"/>
-      </geometry>
-      <origin rpy="0 0 0" xyz="0 0 0"/>
-    </visual>
-    <collision>
-      <geometry>
-        <mesh filename="package://r2_description/meshes/r2c_legs/r2cl_ext_bone2.dae"/>
+      <inertia ixx="0.1" ixy="0.00" ixz="0.0" iyy="0.1" iyz="0.0" izz="0.1"/>
+    </inertial>
+    <visual>
+      <geometry>
+        <mesh filename="package://r2_description/meshes/r2_legs/r2cl_ext_bone2.dae"/>
+      </geometry>
+      <origin rpy="0 0 0" xyz="0 0 0"/>
+    </visual>
+    <collision>
+      <geometry>
+        <mesh filename="package://r2_description/meshes/r2_legs/r2cl_ext_bone2.dae"/>
       </geometry>
       <origin rpy="0 0 0" xyz="0 0 0"/>
@@ -132,20 +129,19 @@
     <dynamics damping="${left_leg_j3_damping}" friction="${left_leg_j3_friction}" />
     <limit effort="330.0" lower="-0.0872664" upper="2.6703515" velocity="1.0"/>
-    <traits spring_k="2.5"   />
   </joint>
   <link name="${robot_name}left_knee">
     <inertial>
       <mass value="4.78221"/>
-      <inertia ixx="0.01671" ixy="0.02240" ixz="-0.00120" iyy="0.07877" iyz="0.00049" izz="0.08739"/>
-    </inertial>
-    <visual>
-      <geometry>
-        <mesh filename="package://r2_description/meshes/r2c_legs/r2cl_ext_bone1.dae"/>
-      </geometry>
-      <origin rpy="0 0 0" xyz="0 0 0"/>
-    </visual>
-    <collision>
-      <geometry>
-        <mesh filename="package://r2_description/meshes/r2c_legs/r2cl_ext_bone1.dae"/>
+      <inertia ixx="0.1" ixy="0.00" ixz="0.0" iyy="0.1" iyz="0.0" izz="0.1"/>
+    </inertial>
+    <visual>
+      <geometry>
+        <mesh filename="package://r2_description/meshes/r2_legs/r2cl_ext_bone1.dae"/>
+      </geometry>
+      <origin rpy="0 0 0" xyz="0 0 0"/>
+    </visual>
+    <collision>
+      <geometry>
+        <mesh filename="package://r2_description/meshes/r2_legs/r2cl_ext_bone1.dae"/>
       </geometry>
       <material name="gold"/>
@@ -160,20 +156,19 @@
     <dynamics damping="${left_leg_j4_damping}" friction="${left_leg_j4_friction}" />
     <limit effort="330.0" lower="-4.71239" upper="4.71239" velocity="1.0"/>
-    <traits spring_k="2.5"   />
   </joint>
   <link name="${robot_name}left_lower_leg">
     <inertial>
       <mass value="3.73407"/>
-      <inertia ixx="0.05967" ixy="-0.00299" ixz="0.00939" iyy="0.05554" iyz="0.01276" izz="0.01370"/>
-    </inertial>
-    <visual>
-      <geometry>
-        <mesh filename="package://r2_description/meshes/r2c_legs/r2cl_ext_bone2.dae"/>
-      </geometry>
-      <origin rpy="0 0 0" xyz="0 0 0"/>
-    </visual>
-    <collision>
-      <geometry>
-        <mesh filename="package://r2_description/meshes/r2c_legs/r2cl_ext_bone2.dae"/>
+      <inertia ixx="0.1" ixy="0.00" ixz="0.0" iyy="0.1" iyz="0.0" izz="0.1"/>
+    </inertial>
+    <visual>
+      <geometry>
+        <mesh filename="package://r2_description/meshes/r2_legs/r2cl_ext_bone2.dae"/>
+      </geometry>
+      <origin rpy="0 0 0" xyz="0 0 0"/>
+    </visual>
+    <collision>
+      <geometry>
+        <mesh filename="package://r2_description/meshes/r2_legs/r2cl_ext_bone2.dae"/>
       </geometry>
       <origin rpy="0 0 0" xyz="0 0 0"/>
@@ -187,20 +182,19 @@
     <dynamics damping="${left_leg_j5_damping}" friction="${left_leg_j5_friction}" />
     <limit effort="330.0" lower="-0.0872664" upper="2.6703515" velocity="1.0"/>
-    <traits spring_k="2.5"   />
   </joint>
   <link name="${robot_name}left_ankle_pitch">
     <inertial>
       <mass value="4.78221"/>
-      <inertia ixx="0.01671" ixy="0.02240" ixz="-0.00120" iyy="0.07877" iyz="0.00049" izz="0.08739"/>
-    </inertial>
-    <visual>
-      <geometry>
-        <mesh filename="package://r2_description/meshes/r2c_legs/r2cl_ext_bone1.dae"/>
-      </geometry>
-      <origin rpy="0 0 0" xyz="0 0 0"/>
-    </visual>
-    <collision>
-      <geometry>
-        <mesh filename="package://r2_description/meshes/r2c_legs/r2cl_ext_bone1.dae"/>
+      <inertia ixx="0.1" ixy="0.00" ixz="0.0" iyy="0.1" iyz="0.0" izz="0.1"/>
+    </inertial>
+    <visual>
+      <geometry>
+        <mesh filename="package://r2_description/meshes/r2_legs/r2cl_ext_bone1.dae"/>
+      </geometry>
+      <origin rpy="0 0 0" xyz="0 0 0"/>
+    </visual>
+    <collision>
+      <geometry>
+        <mesh filename="package://r2_description/meshes/r2_legs/r2cl_ext_bone1.dae"/>
       </geometry>
       <origin rpy="0 0 0" xyz="0 0 0"/>
@@ -214,10 +208,9 @@
     <dynamics damping="${left_leg_j6_damping}" friction="${left_leg_j6_friction}" />
     <limit effort="330.0" lower="-4.71239" upper="4.71239" velocity="1.0"/>
-    <traits spring_k="2.5"   />
   </joint>
   <link name="${robot_name}left_ankle_roll">
     <inertial>
       <mass value="1.50471"/>
-      <inertia ixx="0.00203" ixy="0.00003" ixz="0.0" iyy="0.00204" iyz="0.0" izz="0.00335"/>
+      <inertia ixx="0.1" ixy="0.00" ixz="0.0" iyy="0.1" iyz="0.0" izz="0.1"/>
     </inertial>
     <visual>

File: r2_description/urdf/r2_legs/r2_legs.pelvis.xacro (robot description, xacro)
@@ -8,5 +8,5 @@
     <visual>
       <geometry>
-        <mesh filename="package://r2_description/meshes/r2c_legs/r2cl_ext_pelvis.dae"/>
+        <mesh filename="package://r2_description/meshes/r2_legs/r2cl_ext_pelvis.dae"/>
       </geometry>
       <material name="gold"/>
@@ -15,5 +15,5 @@
     <collision>
       <geometry>
-        <mesh filename="package://r2_description/meshes/r2c_legs/r2cl_ext_pelvis.dae"/>
+        <mesh filename="package://r2_description/meshes/r2_legs/r2cl_ext_pelvis.dae"/>
       </geometry>
       <origin xyz="0 0 0" rpy="0 0 0"/>

File: r2_description/urdf/r2_legs/r2_legs.right_foot.xacro (robot description, xacro)
@@ -19,5 +19,5 @@
     <visual>
       <geometry>
-        <mesh filename="package://r2_description/meshes/r2c_legs/r2cl_foot.dae"/>
+        <mesh filename="package://r2_description/meshes/r2_legs/r2cl_foot.dae"/>
       </geometry>
       <material name="gold"/>
@@ -26,5 +26,5 @@
     <collision>
       <geometry>
-        <mesh filename="package://r2_description/meshes/r2c_legs/r2cl_foot.dae"/>
+        <mesh filename="package://r2_description/meshes/r2_legs/r2cl_foot.dae"/>
       </geometry>
       <origin rpy="0 0 0" xyz="0 0 0"/>
@@ -85,9 +85,9 @@
     <inertial>
       <mass value="0.16268"/>
-      <inertia ixx="0.001" ixy="0.0" ixz="0.0" iyy="0.001" iyz="0.0" izz="0.001"/>
+      <inertia ixx="0.1" ixy="0.0" ixz="0.0" iyy="0.1" iyz="0.0" izz="0.1"/>
     </inertial>
     <visual>
       <geometry>
-        <mesh filename="package://r2_description/meshes/r2c_legs/r2cl_foot_jaw1.dae"/>
+        <mesh filename="package://r2_description/meshes/r2_legs/r2cl_foot_jaw1.dae"/>
       </geometry>
       <origin rpy="0 0 0" xyz="0 0 0"/>
@@ -95,5 +95,5 @@
     <collision>
       <geometry>
-        <mesh filename="package://r2_description/meshes/r2c_legs/r2cl_foot_jaw1.dae"/>
+        <mesh filename="package://r2_description/meshes/r2_legs/r2cl_foot_jaw1.dae"/>
       </geometry>
       <origin rpy="0 0 0" xyz="0 0 0"/>
@@ -103,9 +103,9 @@
     <inertial>
       <mass value="0.16268"/>
-      <inertia ixx="0.001" ixy="0.0" ixz="0.0" iyy="0.001" iyz="0.0" izz="0.001"/>
+      <inertia ixx="0.1" ixy="0.0" ixz="0.0" iyy="0.1" iyz="0.0" izz="0.1"/>
     </inertial>
     <visual>
       <geometry>
-        <mesh filename="package://r2_description/meshes/r2c_legs/r2cl_foot_jaw2.dae"/>
+        <mesh filename="package://r2_description/meshes/r2_legs/r2cl_foot_jaw2.dae"/>
       </geometry>
       <origin rpy="0 0 0" xyz="0 0 0"/>
@@ -113,5 +113,5 @@
     <collision>
       <geometry>
-        <mesh filename="package://r2_description/meshes/r2c_legs/r2cl_foot_jaw2.dae"/>
+        <mesh filename="package://r2_description/meshes/r2_legs/r2cl_foot_jaw2.dae"/>
       </geometry>
       <origin rpy="0 0 0" xyz="0 0 0"/>

File: r2_description/urdf/r2_legs/r2_legs.right_leg.xacro (robot description, xacro)
@@ -56,9 +56,9 @@
     <inertial>
       <mass value="2.33931"/>
-      <inertia ixx="0.02547" ixy="0.00297" ixz="-0.00847" iyy="0.02956" iyz="0.00636" izz="0.01148"/>
-    </inertial>
-    <visual>
-      <geometry>
-        <mesh filename="package://r2_description/meshes/r2c_legs/r2cl_ext_bone3.dae"/>
+      <inertia ixx="0.1" ixy="0.00" ixz="0.0" iyy="0.1" iyz="0.0" izz="0.1"/>
+    </inertial>
+    <visual>
+      <geometry>
+        <mesh filename="package://r2_description/meshes/r2_legs/r2cl_ext_bone3.dae"/>
       </geometry>
       <origin rpy="0 0 0" xyz="0.0 0.0 0.0"/>
@@ -66,5 +66,5 @@
     <collision>
       <geometry>
-        <mesh filename="package://r2_description/meshes/r2c_legs/r2cl_ext_bone3.dae"/>
+        <mesh filename="package://r2_description/meshes/r2_legs/r2cl_ext_bone3.dae"/>
       </geometry>
       <origin rpy="0 0 0" xyz="0.0 0.0 0.0"/>
@@ -83,15 +83,15 @@
     <inertial>
       <mass value="4.78221"/>
-      <inertia ixx="0.01671" ixy="0.02240" ixz="-0.00120" iyy="0.07877" iyz="0.00049" izz="0.08739"/>
-    </inertial>
-    <visual>
-      <geometry>
-        <mesh filename="package://r2_description/meshes/r2c_legs/r2cl_ext_bone1.dae"/>
-      </geometry>
-      <origin rpy="0 0 0" xyz="0 0 0"/>
-    </visual>
-    <collision>
-      <geometry>
-        <mesh filename="package://r2_description/meshes/r2c_legs/r2cl_ext_bone1.dae"/>
+      <inertia ixx="0.1" ixy="0.00" ixz="0.0" iyy="0.1" iyz="0.0" izz="0.1"/>
+    </inertial>
+    <visual>
+      <geometry>
+        <mesh filename="package://r2_description/meshes/r2_legs/r2cl_ext_bone1.dae"/>
+      </geometry>
+      <origin rpy="0 0 0" xyz="0 0 0"/>
+    </visual>
+    <collision>
+      <geometry>
+        <mesh filename="package://r2_description/meshes/r2_legs/r2cl_ext_bone1.dae"/>
       </geometry>
       <origin rpy="0 0 0" xyz="0 0 0"/>
@@ -110,15 +110,15 @@
     <inertial>
       <mass value="3.73407"/>
-      <inertia ixx="0.05967" ixy="-0.00299" ixz="0.00939" iyy="0.05554" iyz="0.01276" izz="0.01370"/>
-    </inertial>
-    <visual>
-      <geometry>
-        <mesh filename="package://r2_description/meshes/r2c_legs/r2cl_ext_bone2.dae"/>
-      </geometry>
-      <origin rpy="0 0 0" xyz="0 0 0"/>
-    </visual>
-    <collision>
-      <geometry>
-        <mesh filename="package://r2_description/meshes/r2c_legs/r2cl_ext_bone2.dae"/>
+      <inertia ixx="0.1" ixy="0.00" ixz="0.0" iyy="0.1" iyz="0.0" izz="0.1"/>
+    </inertial>
+    <visual>
+      <geometry>
+        <mesh filename="package://r2_description/meshes/r2_legs/r2cl_ext_bone2.dae"/>
+      </geometry>
+      <origin rpy="0 0 0" xyz="0 0 0"/>
+    </visual>
+    <collision>
+      <geometry>
+        <mesh filename="package://r2_description/meshes/r2_legs/r2cl_ext_bone2.dae"/>
       </geometry>
       <origin rpy="0 0 0" xyz="0 0 0.0"/>
@@ -137,15 +137,15 @@
     <inertial>
       <mass value="4.78221"/>
-      <inertia ixx="0.01671" ixy="0.02240" ixz="-0.00120" iyy="0.07877" iyz="0.00049" izz="0.08739"/>
-    </inertial>
-    <visual>
-      <geometry>
-        <mesh filename="package://r2_description/meshes/r2c_legs/r2cl_ext_bone1.dae"/>
-      </geometry>
-      <origin rpy="0 0 0" xyz="0 0 0"/>
-    </visual>
-    <collision>
-      <geometry>
-        <mesh filename="package://r2_description/meshes/r2c_legs/r2cl_ext_bone1.dae"/>
+      <inertia ixx="0.1" ixy="0.00" ixz="0.0" iyy="0.1" iyz="0.0" izz="0.1"/>
+    </inertial>
+    <visual>
+      <geometry>
+        <mesh filename="package://r2_description/meshes/r2_legs/r2cl_ext_bone1.dae"/>
+      </geometry>
+      <origin rpy="0 0 0" xyz="0 0 0"/>
+    </visual>
+    <collision>
+      <geometry>
+        <mesh filename="package://r2_description/meshes/r2_legs/r2cl_ext_bone1.dae"/>
       </geometry>
       <material name="gold"/>
@@ -165,15 +165,15 @@
     <inertial>
       <mass value="3.73407"/>
-      <inertia ixx="0.05967" ixy="-0.00299" ixz="0.00939" iyy="0.05554" iyz="0.01276" izz="0.01370"/>
-    </inertial>
-    <visual>
-      <geometry>
-        <mesh filename="package://r2_description/meshes/r2c_legs/r2cl_ext_bone2.dae"/>
-      </geometry>
-      <origin rpy="0 0 0" xyz="0 0 0"/>
-    </visual>
-    <collision>
-      <geometry>
-        <mesh filename="package://r2_description/meshes/r2c_legs/r2cl_ext_bone2.dae"/>
+      <inertia ixx="0.1" ixy="0.00" ixz="0.0" iyy="0.1" iyz="0.0" izz="0.1"/>
+    </inertial>
+    <visual>
+      <geometry>
+        <mesh filename="package://r2_description/meshes/r2_legs/r2cl_ext_bone2.dae"/>
+      </geometry>
+      <origin rpy="0 0 0" xyz="0 0 0"/>
+    </visual>
+    <collision>
+      <geometry>
+        <mesh filename="package://r2_description/meshes/r2_legs/r2cl_ext_bone2.dae"/>
       </geometry>
       <origin rpy="0 0 0" xyz="0 0 0.0"/>
@@ -192,15 +192,15 @@
     <inertial>
       <mass value="4.78221"/>
-      <inertia ixx="0.01671" ixy="0.02240" ixz="-0.00120" iyy="0.07877" iyz="0.00049" izz="0.08739"/>
-    </inertial>
-    <visual>
-      <geometry>
-        <mesh filename="package://r2_description/meshes/r2c_legs/r2cl_ext_bone1.dae"/>
-      </geometry>
-      <origin rpy="0 0 0" xyz="0 0 0"/>
-    </visual>
-    <collision>
-      <geometry>
-        <mesh filename="package://r2_description/meshes/r2c_legs/r2cl_ext_bone1.dae"/>
+      <inertia ixx="0.1" ixy="0.00" ixz="0.0" iyy="0.1" iyz="0.0" izz="0.1"/>
+    </inertial>
+    <visual>
+      <geometry>
+        <mesh filename="package://r2_description/meshes/r2_legs/r2cl_ext_bone1.dae"/>
+      </geometry>
+      <origin rpy="0 0 0" xyz="0 0 0"/>
+    </visual>
+    <collision>
+      <geometry>
+        <mesh filename="package://r2_description/meshes/r2_legs/r2cl_ext_bone1.dae"/>
       </geometry>
       <origin rpy="0 0 0" xyz="0 0 0"/>
@@ -219,5 +219,5 @@
     <inertial>
       <mass value="1.50471"/>
-      <inertia ixx="0.00203" ixy="0.00003" ixz="0.0" iyy="0.00204" iyz="0.0" izz="0.00335"/>
+      <inertia ixx="0.1" ixy="0.00" ixz="0.0" iyy="0.1" iyz="0.0" izz="0.1"/>
     </inertial>
     <visual>
