Commit message: fixed geometry models for body, cover, and shoulder to not always be in collision. regenerate teh moveit stuff to take advantage of this, it should work better now.

File: r2_description/urdf/r2.body.xacro (robot description, xacro)
@@ -16,12 +16,12 @@
          <mesh filename="package://r2_description/meshes/Body.dae"/>
       </geometry>
-      <origin rpy="-1.57 0 -1.57" xyz="0.02 0.05 -0.5625"/>
+      <origin rpy="-1.57 0 -1.57" xyz="0.01 0.05 -0.5625"/>
     </visual>
-    <collision>
+    <!-- <collision>
       <geometry>
          <mesh filename="package://r2_description/meshes/Body.dae"/>
       </geometry>
-      <origin rpy="-1.57 0 -1.57" xyz="0.02 0.05 -0.5625"/>
-    </collision>
+      <origin rpy="-1.57 0 -1.57" xyz="0.00 0.05 -0.5625"/>
+    </collision> -->
     <inertial>
       <mass value="10"/>
@@ -55,5 +55,6 @@
          <mesh filename="package://r2_description/meshes/Body_Cover.dae"/>
       </geometry>
-      <origin rpy="-1.57 0 -1.57" xyz="0.02 0.05 -0.5625"/>
+<!--       <origin rpy="-1.57 0 -1.57" xyz="0.02 0.05 -0.5625"/>
+ -->      <origin rpy="-1.57 0 -1.57" xyz="0.01 0.05 -0.5625"/>
     </visual>
     <collision>
@@ -61,5 +62,5 @@
          <mesh filename="package://r2_description/meshes/Body_Cover.dae"/>
       </geometry>
-      <origin rpy="-1.57 0 -1.57" xyz="0.02 0.05 -0.5625"/>
+      <origin rpy="-1.57 0 -1.57" xyz="0.01 0.05 -0.5625"/>
     </collision>
     <inertial>

File: r2_description/urdf/r2.left_arm.xacro (robot description, xacro)
@@ -31,10 +31,10 @@
       <origin rpy="0 0 1.57" xyz="0 0 .08"/>
     </visual>
-    <collision>
-      <geometry>
-        <mesh filename="package://r2_description/meshes/Left_Shoulder_Upper.dae"/>
+    <!-- <collision>
+      <geometry>
+        <mesh filename="package://r2_description/meshes/Left_Shoulder_Upper.dae" scale="0.7 0.7 0.7"/>
       </geometry>
       <origin rpy="0 0 1.57" xyz="0 0 .08"/>
-    </collision>
+    </collision> -->
     <inertial>
 	<origin xyz="-0.0089916 -0.00131572   0.10287   "/>
@@ -59,10 +59,10 @@
       <origin rpy=".0 0 -1.57" xyz="0 0 0"/>
     </visual>
-    <collision>
+    <!-- <collision>
       <geometry>
         <mesh filename="package://r2_description/meshes/Left_Shoulder_Lower.dae"/>
       </geometry>
       <origin rpy=".0 0 -1.57" xyz="0 0 0"/>
-    </collision>
+    </collision> -->
      <inertial>
         <origin xyz="0.037084 -0.00028448   0.0077978   "/>
@@ -89,5 +89,5 @@
     <collision>
       <geometry>
-        <mesh filename="package://r2_description/meshes/Left_Upper_Arm.dae"/>
+        <mesh filename="package://r2_description/meshes/Left_Upper_Arm.dae" scale="0.8 0.8 0.8"/>
       </geometry>
       <origin rpy="0 0 3.14" xyz="0 0 .1016"/>

File: r2_description/urdf/r2.right_arm.xacro (robot description, xacro)
@@ -31,10 +31,10 @@
       <origin rpy="0 0 2.25" xyz="0 0 .0254"/>
     </visual>
-    <collision>
+    <!-- <collision>
       <geometry>
         <mesh filename="package://r2_description/meshes/Right_Shoulder_Upper.dae"/>
       </geometry>
       <origin rpy="0 0 2.35" xyz="0 0 .0254"/>
-    </collision>
+    </collision> -->
     <inertial>
         <origin xyz="0.0089916 -0.00131572  0.10287"/>
@@ -59,10 +59,10 @@
       <origin rpy=".0 0 1.57" xyz="0 0 0"/>
     </visual>
-    <collision>
+  <!--   <collision>
       <geometry>
         <mesh filename="package://r2_description/meshes/Right_Shoulder_Lower.dae"/>
       </geometry>
       <origin rpy=".0 0 1.57" xyz="0 0 0"/>
-    </collision>
+    </collision> -->
      <inertial>
         <origin xyz="0.0077978 0.037084 0.00028448"/>
