Commit message: updated to latest nasa version

File: r2_description/urdf/r2.head.xacro (robot description, xacro)
@@ -7,4 +7,6 @@
   <property name="neck_j2_damping" value= "10.0" />
   <property name="neck_j2_friction" value= "0.0" />
+  <property name="effort_limit" value= "10000.0" />
+  <property name="velocity_limit" value= "1000.0" />
   <joint name="${robot_name}neck/joint0" type="revolute">
     <parent link="${robot_name}waist_center"/>
@@ -13,5 +15,5 @@
     <dynamics damping="${neck_j0_damping}" friction="${neck_j0_friction}"/>
     <axis xyz="0 0 1"/>
-    <limit effort="100000.0" lower="-0.7" upper="0.175" velocity="1000"/>
+    <limit effort="${effort_limit}" lower="-0.7" upper="0.175" velocity="${velocity_limit}"/>
   </joint>
   <link name="${robot_name}neck_base">
@@ -39,5 +41,5 @@
     <dynamics damping="${neck_j1_damping}" friction="${neck_j1_friction}"/>
     <axis xyz="0 0 1"/>
-    <limit effort="100000.0" lower="-1.22" upper="1.22" velocity="1000"/>
+    <limit effort="${effort_limit}" lower="-1.22" upper="1.22" velocity="${velocity_limit}"/>
   </joint>
   <link name="${robot_name}neck_lower_pitch">
@@ -65,5 +67,5 @@
     <dynamics damping="${neck_j2_damping}" friction="${neck_j2_friction}"/>
     <axis xyz="0 0 1"/>
-    <limit effort="100000.0" lower="-0.7" upper="0.175" velocity="1000"/>
+    <limit effort="${effort_limit}" lower="-0.7" upper="0.175" velocity="${velocity_limit}"/>
   </joint>
   <link name="${robot_name}neck_roll">

Commit message: added asus and camera to moveit rviz. added more head poses

File: r2_description/urdf/r2.head.xacro (robot description, xacro)
@@ -105,9 +105,17 @@
 <!-- ORIGINAL     <origin rpy="1.57 0 1.57 " xyz="0.066675 -0.0508 -0.116205 "/>  -->
   </joint>
-  <joint name="${robot_name}fixed/neck_upper_pitch/simulated_asus_frame" type="fixed">
-    <parent link="${robot_name}neck_upper_pitch"/>
-    <child link="${robot_name}simulated_asus_frame"/>
-    <dynamics damping="1.0" />
-    <origin rpy="0 0 0" xyz="0.12 -0.015 -0.14 "/>
+  <joint name="${robot_name}fixed/neck_upper_pitch/simulated_asus_camera_frame" type="fixed">
+    <parent link="${robot_name}neck_upper_pitch"/>
+    <child link="${robot_name}simulated_asus_camera_frame"/>
+    <dynamics damping="1.0" />
+    <origin rpy="3.14 0 0" xyz="0.12 -0.015 -0.14 "/>
+<!--     <origin rpy="0 0 0" xyz="0.12 -0.015 -0.14 "/> -->
+  </joint>
+  <joint name="${robot_name}fixed/neck_upper_pitch/simulated_asus_depth_frame" type="fixed">
+    <parent link="${robot_name}neck_upper_pitch"/>
+    <child link="${robot_name}simulated_asus_depth_frame"/>
+    <dynamics damping="1.0" />
+    <origin rpy="1.57 0 1.57" xyz="0.12 -0.015 -0.14 "/>
+<!--     <origin rpy="0 0 0" xyz="0.12 -0.015 -0.14 "/> -->
   </joint>
   <joint name="${robot_name}fixed/neck_upper_pitch/vision_center_frame" type="fixed">
@@ -137,5 +145,12 @@
   </link>
  <!-- simulated asus -->
- <link name="${robot_name}simulated_asus_frame">
+ <link name="${robot_name}simulated_asus_camera_frame">
+    <inertial>
+      <mass value=".01"/>
+      <inertia ixx=".0010" ixy="0.0" ixz="0.0" iyy=".0010" iyz="0.0" izz=".0010"/>
+    </inertial>
+  </link>
+  <!-- simulated asus -->
+ <link name="${robot_name}simulated_asus_depth_frame">
     <inertial>
       <mass value=".01"/>
