Commit message: MIMIC tags

File: r2_description/urdf/r2.left_hand.xacro (robot description, xacro)
@@ -276,4 +276,5 @@
     <limit effort="10000000.0" lower="0.0" upper="1.57" velocity="1000"/>
     <dynamics damping="${left_arm_hand_index_j3_damping}" friction="${left_arm_hand_index_j3_friction}"/>
+    <mimic joint="${robot_name}left_arm/hand/index/joint2"/>
   </joint>
   <link name="${robot_name}left_index_distal">
@@ -377,4 +378,5 @@
     <limit effort="10000000.0" lower="0.0" upper="1.57" velocity="1000"/>
     <dynamics damping="${left_arm_hand_middle_j3_damping}" friction="${left_arm_hand_middle_j3_friction}"/>
+    <mimic joint="${robot_name}left_arm/hand/middle/joint2"/>
   </joint>
   <link name="${robot_name}left_middle_distal">
@@ -432,4 +434,5 @@
     <limit effort="10000000.0" lower="0" upper="2.9671" velocity="1000"/>
     <dynamics damping="${left_arm_hand_ring_j1_damping}" friction="${left_arm_hand_ring_j1_friction}"/>
+    <mimic joint="${robot_name}left_arm/hand/ring/joint0"/>
   </joint>
   <link name="${robot_name}left_ring_medial">
@@ -458,4 +461,5 @@
     <limit effort="10000000.0" lower="0" upper="2.9671" velocity="1000"/>
     <dynamics damping="${left_arm_hand_ring_j2_damping}" friction="${left_arm_hand_ring_j2_friction}"/>
+    <mimic joint="${robot_name}left_arm/hand/ring/joint0"/>
   </joint>
   <link name="${robot_name}left_ring_distal">
@@ -513,4 +517,5 @@
     <limit effort="10000000.0" lower="0" upper="2.9671" velocity="1000"/>
     <dynamics damping="${left_arm_hand_little_j1_damping}" friction="${left_arm_hand_little_j1_friction}"/>
+    <mimic joint="${robot_name}left_arm/hand/little/joint0"/>
   </joint>
   <link name="${robot_name}left_little_medial">
@@ -539,4 +544,5 @@
     <limit effort="10000000.0" lower="0" upper="2.9671" velocity="1000"/>
     <dynamics damping="${left_arm_hand_little_j2_damping}" friction="${left_arm_hand_little_j2_friction}"/>
+    <mimic joint="${robot_name}left_arm/hand/little/joint0"/>
   </joint>
   <link name="${robot_name}left_little_distal">

File: r2_description/urdf/r2.right_hand.xacro (robot description, xacro)
@@ -276,4 +276,5 @@
     <limit effort="10000000.0" lower="0.0" upper="1.57" velocity="1000"/>
     <dynamics damping="${right_arm_hand_index_j3_damping}" friction="${right_arm_hand_index_j3_friction}"/>
+    <mimic joint="${robot_name}right_arm/hand/index/joint2"/>
   </joint>
   <link name="${robot_name}right_index_distal">
@@ -377,4 +378,5 @@
     <limit effort="10000000.0" lower="0.0" upper="1.57" velocity="1000"/>
     <dynamics damping="${right_arm_hand_middle_j3_damping}" friction="${right_arm_hand_middle_j3_friction}"/>
+    <mimic joint="${robot_name}right_arm/hand/middle/joint2"/>
   </joint>
   <link name="${robot_name}right_middle_distal">
@@ -432,4 +434,5 @@
     <limit effort="10000000.0" lower="0" upper="2.9671" velocity="1000"/>
     <dynamics damping="${right_arm_hand_ring_j1_damping}" friction="${right_arm_hand_ring_j1_friction}"/>
+    <mimic joint="${robot_name}right_arm/hand/ring/joint0"/>
   </joint>
   <link name="${robot_name}right_ring_medial">
@@ -458,4 +461,5 @@
     <limit effort="10000000.0" lower="0" upper="2.9671" velocity="1000"/>
     <dynamics damping="${right_arm_hand_ring_j2_damping}" friction="${right_arm_hand_ring_j2_friction}"/>
+    <mimic joint="${robot_name}right_arm/hand/ring/joint0"/>
   </joint>
   <link name="${robot_name}right_ring_distal">
@@ -513,4 +517,5 @@
     <limit effort="10000000.0" lower="0" upper="2.9671" velocity="1000"/>
     <dynamics damping="${right_arm_hand_little_j1_damping}" friction="${right_arm_hand_little_j1_friction}"/>
+    <mimic joint="${robot_name}right_arm/hand/little/joint0"/>
   </joint>
   <link name="${robot_name}right_little_medial">
@@ -539,4 +544,5 @@
     <limit effort="10000000.0" lower="0" upper="2.9671" velocity="1000"/>
     <dynamics damping="${right_arm_hand_little_j2_damping}" friction="${right_arm_hand_little_j2_friction}"/>
+    <mimic joint="${robot_name}right_arm/hand/little/joint0"/>
   </joint>
   <link name="${robot_name}right_little_distal">

Commit message: No mimic

File: r2_description/urdf/r2.left_hand.xacro (robot description, xacro)
@@ -276,5 +276,4 @@
     <limit effort="10000000.0" lower="0.0" upper="1.57" velocity="1000"/>
     <dynamics damping="${left_arm_hand_index_j3_damping}" friction="${left_arm_hand_index_j3_friction}"/>
-    <mimic joint="${robot_name}left_arm/hand/index/joint2"/>
   </joint>
   <link name="${robot_name}left_index_distal">
@@ -378,5 +377,4 @@
     <limit effort="10000000.0" lower="0.0" upper="1.57" velocity="1000"/>
     <dynamics damping="${left_arm_hand_middle_j3_damping}" friction="${left_arm_hand_middle_j3_friction}"/>
-    <mimic joint="${robot_name}left_arm/hand/middle/joint2"/>
   </joint>
   <link name="${robot_name}left_middle_distal">
@@ -434,5 +432,4 @@
     <limit effort="10000000.0" lower="0" upper="2.9671" velocity="1000"/>
     <dynamics damping="${left_arm_hand_ring_j1_damping}" friction="${left_arm_hand_ring_j1_friction}"/>
-    <mimic joint="${robot_name}left_arm/hand/ring/joint0"/>
   </joint>
   <link name="${robot_name}left_ring_medial">
@@ -461,5 +458,4 @@
     <limit effort="10000000.0" lower="0" upper="2.9671" velocity="1000"/>
     <dynamics damping="${left_arm_hand_ring_j2_damping}" friction="${left_arm_hand_ring_j2_friction}"/>
-    <mimic joint="${robot_name}left_arm/hand/ring/joint0"/>
   </joint>
   <link name="${robot_name}left_ring_distal">
@@ -517,5 +513,4 @@
     <limit effort="10000000.0" lower="0" upper="2.9671" velocity="1000"/>
     <dynamics damping="${left_arm_hand_little_j1_damping}" friction="${left_arm_hand_little_j1_friction}"/>
-    <mimic joint="${robot_name}left_arm/hand/little/joint0"/>
   </joint>
   <link name="${robot_name}left_little_medial">
@@ -544,5 +539,4 @@
     <limit effort="10000000.0" lower="0" upper="2.9671" velocity="1000"/>
     <dynamics damping="${left_arm_hand_little_j2_damping}" friction="${left_arm_hand_little_j2_friction}"/>
-    <mimic joint="${robot_name}left_arm/hand/little/joint0"/>
   </joint>
   <link name="${robot_name}left_little_distal">

File: r2_description/urdf/r2.right_hand.xacro (robot description, xacro)
@@ -276,5 +276,4 @@
     <limit effort="10000000.0" lower="0.0" upper="1.57" velocity="1000"/>
     <dynamics damping="${right_arm_hand_index_j3_damping}" friction="${right_arm_hand_index_j3_friction}"/>
-    <mimic joint="${robot_name}right_arm/hand/index/joint2"/>
   </joint>
   <link name="${robot_name}right_index_distal">
@@ -378,5 +377,4 @@
     <limit effort="10000000.0" lower="0.0" upper="1.57" velocity="1000"/>
     <dynamics damping="${right_arm_hand_middle_j3_damping}" friction="${right_arm_hand_middle_j3_friction}"/>
-    <mimic joint="${robot_name}right_arm/hand/middle/joint2"/>
   </joint>
   <link name="${robot_name}right_middle_distal">
@@ -434,5 +432,4 @@
     <limit effort="10000000.0" lower="0" upper="2.9671" velocity="1000"/>
     <dynamics damping="${right_arm_hand_ring_j1_damping}" friction="${right_arm_hand_ring_j1_friction}"/>
-    <mimic joint="${robot_name}right_arm/hand/ring/joint0"/>
   </joint>
   <link name="${robot_name}right_ring_medial">
@@ -461,5 +458,4 @@
     <limit effort="10000000.0" lower="0" upper="2.9671" velocity="1000"/>
     <dynamics damping="${right_arm_hand_ring_j2_damping}" friction="${right_arm_hand_ring_j2_friction}"/>
-    <mimic joint="${robot_name}right_arm/hand/ring/joint0"/>
   </joint>
   <link name="${robot_name}right_ring_distal">
@@ -517,5 +513,4 @@
     <limit effort="10000000.0" lower="0" upper="2.9671" velocity="1000"/>
     <dynamics damping="${right_arm_hand_little_j1_damping}" friction="${right_arm_hand_little_j1_friction}"/>
-    <mimic joint="${robot_name}right_arm/hand/little/joint0"/>
   </joint>
   <link name="${robot_name}right_little_medial">
@@ -544,5 +539,4 @@
     <limit effort="10000000.0" lower="0" upper="2.9671" velocity="1000"/>
     <dynamics damping="${right_arm_hand_little_j2_damping}" friction="${right_arm_hand_little_j2_friction}"/>
-    <mimic joint="${robot_name}right_arm/hand/little/joint0"/>
   </joint>
   <link name="${robot_name}right_little_distal">
