Commit message: changed link root of legs and inertial props of feet

File: r2_description/urdf/r2_legs/r2_legs.left_foot.xacro (robot description, xacro)
@@ -15,5 +15,5 @@
     <inertial>
       <mass value="4.40475"/>
-      <inertia ixx="0.04809" ixy="0.00026" ixz="0.00038" iyy="0.04403" iyz="-0.00321" izz="0.0127"/>
+      <inertia ixx="0.1" ixy="0.0" ixz="0.0" iyy="0.1" iyz="0.0" izz="0.1"/>
     </inertial>
     <visual>
@@ -21,5 +21,5 @@
         <mesh filename="package://r2_description/meshes/r2_legs/r2cl_foot.dae"/>
       </geometry>
-      <origin rpy="0 0 0" xyz="0 0 0"/>
+      <origin xyz="0 0 0" rpy="0 0 0" />
     </visual>
     <collision>

File: r2_description/urdf/r2_legs/r2_legs.right_foot.xacro (robot description, xacro)
@@ -15,5 +15,5 @@
     <inertial>
       <mass value="4.40475"/>
-      <inertia ixx="0.04809" ixy="0.00026" ixz="0.00038" iyy="0.04403" iyz="-0.00321" izz="0.0127"/>
+       <inertia ixx="0.1" ixy="0.0" ixz="0.0" iyy="0.1" iyz="0.0" izz="0.1"/>
     </inertial>
     <visual>
@@ -22,5 +22,5 @@
       </geometry>
       <material name="gold"/>
-      <origin rpy="0 0 0" xyz="0 0 0"/>
+      <origin xyz="0 0 0" rpy="0 0 0" />
     </visual>
     <collision>

Commit message: modifed rviz config for sensors. added frames in model for simualted Camboard nanons on feet.

File: r2_description/urdf/r2_legs/r2_legs.left_foot.xacro (robot description, xacro)
@@ -30,4 +30,16 @@
     </collision>
   </link>
+  <joint name="${robot_name}fixed/left_foot/simulated_camboard" type="fixed">
+    <parent link="${robot_name}left_leg_foot"/>
+    <child link="${robot_name}simulated_left_foot_camboard_frame"/>
+    <dynamics damping="1.0" />
+    <origin rpy="0 -1.57 -1.57" xyz="0.015 0.07 .165"/>
+  </joint>
+  <joint name="${robot_name}fixed/left_foot/simulated_camboard_depth" type="fixed">
+    <parent link="${robot_name}left_leg_foot"/>
+    <child link="${robot_name}simulated_left_foot_camboard_depth_frame"/>
+    <dynamics damping="1.0" />
+    <origin rpy="3.14 3.14 0" xyz="0.015 0.07 .165"/>
+  </joint>
 <!--  placeholder for screw joint-->
   <joint name="${robot_name}left_leg/gripper/joint0" type="revolute">
@@ -79,4 +91,18 @@
   <non_visual_link name="${robot_name}left_hr_tip"/>
   <non_visual_link name="${robot_name}left_st_tip"/>
+ <!-- simulated camboard -->
+  <link name="${robot_name}simulated_left_foot_camboard_frame">
+    <inertial>
+      <mass value=".1"/>
+      <inertia ixx=".01" ixy="0.0" ixz="0.0" iyy=".01" iyz="0.0" izz=".01"/>
+    </inertial>
+  </link>
+  <!-- simulated camboard -->
+  <link name="${robot_name}simulated_left_foot_camboard_depth_frame">
+    <inertial>
+      <mass value=".1"/>
+      <inertia ixx=".01" ixy="0.0" ixz="0.0" iyy=".01" iyz="0.0" izz=".01"/>
+    </inertial>
+  </link>
   <link name="${robot_name}left_leg_jaw0">
     <inertial>

File: r2_description/urdf/r2_legs/r2_legs.right_foot.xacro (robot description, xacro)
@@ -31,4 +31,16 @@
     </collision>
   </link>
+  <joint name="${robot_name}fixed/right_foot/simulated_camboard" type="fixed">
+    <parent link="${robot_name}right_leg_foot"/>
+    <child link="${robot_name}simulated_right_foot_camboard_frame"/>
+    <dynamics damping="1.0" />
+    <origin rpy="0 -1.57 -1.57" xyz="0.015 0.07 .165"/>
+  </joint>
+  <joint name="${robot_name}fixed/right_foot/simulated_camboard_depth" type="fixed">
+    <parent link="${robot_name}right_leg_foot"/>
+    <child link="${robot_name}simulated_right_foot_camboard_depth_frame"/>
+    <dynamics damping="1.0" />
+    <origin rpy="3.14 3.14 0" xyz="0.015 0.07 .165"/>
+  </joint>
 <!--  placeholder for screw joint-->
   <joint name="${robot_name}right_leg/gripper/joint0" type="prismatic">
@@ -82,4 +94,18 @@
   <non_visual_link name="${robot_name}right_hr_tip"/>
   <non_visual_link name="${robot_name}right_st_tip"/>
+  <!-- simulated camboard -->
+  <link name="${robot_name}simulated_right_foot_camboard_frame">
+    <inertial>
+      <mass value=".1"/>
+      <inertia ixx=".01" ixy="0.0" ixz="0.0" iyy=".01" iyz="0.0" izz=".01"/>
+    </inertial>
+  </link>
+  <!-- simulated camboard -->
+  <link name="${robot_name}simulated_right_foot_camboard_depth_frame">
+    <inertial>
+      <mass value=".1"/>
+      <inertia ixx=".01" ixy="0.0" ixz="0.0" iyy=".01" iyz="0.0" izz=".01"/>
+    </inertial>
+  </link>
   <link name="${robot_name}right_leg_jaw0">
     <inertial>
